File: schematic/oneeye.kicad_sch (KiCad schematic)
At the start: 13 parts, among them J1 Conn_01x03_Pin, J2 Conn_01x02_Pin, J3 Conn_01x02_Pin, M1 Motor_Servo_JR, M2 Motor_Servo_JR, M3 Motor_Servo_JR, M4 Motor_Servo_JR, Q1 2n2222, Q2 2n2222

Commit message: Add files via upload
Connections:
- net at U1.15 (io16): no longer J3.2 (Pin_2)
- net at U1.7 (io2): now also J3.2 (Pin_2)
Other:
- note added: "Note1: io2 is connected to the flash led on the esp32-cam"
- note added: "Note2: io16 is connected to the CS of the video ram, do not use !"
Changed lines of the file:
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@@
-	(wire
-		(pts
-			(xy 128.016 89.408) (xy 128.016 86.36)
-		)
-		(stroke
-			(width 0)
-			(type default)
-		)
-	)
 	(wire
 		(pts
@@
 	(wire
 		(pts
-			(xy 123.698 89.408) (xy 128.016 89.408)
-		)
-		(stroke
-			(width 0)
-			(type default)
-		)
-	)
-	(wire
-		(pts
 			(xy 99.314 124.46) (xy 84.836 124.46)
 		)
@@
 	(wire
 		(pts
+			(xy 131.318 86.36) (xy 131.318 112.014)
+		)
+		(stroke
+			(width 0)
+			(type default)
+		)
+	)
+	(wire
+		(pts
 			(xy 106.172 86.868) (xy 105.918 86.868)
 		)
@@
 	(wire
 		(pts
+			(xy 104.648 112.014) (xy 104.648 102.108)
+		)
+		(stroke
+			(width 0)
+			(type default)
+		)
+	)
+	(wire
+		(pts
+			(xy 131.318 112.014) (xy 104.648 112.014)
+		)
+		(stroke
+			(width 0)
+			(type default)
+		)
+	)
+	(wire
+		(pts
 			(xy 123.444 91.948) (xy 123.698 91.948)
 		)
@@
 	(wire
 		(pts
-			(xy 128.016 86.36) (xy 132.842 86.36)
-		)
-		(stroke
-			(width 0)
-			(type default)
-		)
-	)
-	(wire
-		(pts
 			(xy 117.602 85.598) (xy 117.856 85.598)
 		)
@@
 	(wire
 		(pts
+			(xy 132.842 86.36) (xy 131.318 86.36)
+		)
+		(stroke
+			(width 0)
+			(type default)
+		)
+	)
+	(wire
+		(pts
 			(xy 128.016 67.818) (xy 128.016 83.058)
 		)
@@
 	(wire
 		(pts
+			(xy 104.648 102.108) (xy 105.918 102.108)
+		)
+		(stroke
+			(width 0)
+			(type default)
+		)
+	)
+	(wire
+		(pts
 			(xy 105.918 57.658) (xy 110.998 57.658)
 		)
@@
 		)
 	)
+	(text "Note1: io2 is connected to the flash led on the esp32-cam"
+		(exclude_from_sim no)
+		(at 137.922 116.586 0)
+		(effects
+			(font
+				(size 1.27 1.27)
+			)
+		)
+	)
 	(text "esp32-cam"
 		(exclude_from_sim no)
@@
 		(effects
 			(font
+				(size 1.27 1.27)
+			)
+		)
+	)
+	(text "Note2: io16 is connected to the CS of the video ram, do not use !"
+		(exclude_from_sim no)
+		(at 141.224 119.888 0)
+		(effects
+			(font
